Commit message: drive robot using libgazebo_ros_diff_drive
remove joint_state_publisher_gui from launch file

change lidar joint type to fixed

add comment for controlling the robot

File: src/my_robot/description/gazebo.xacro (robot description, xacro)
@@ -6,4 +6,6 @@
     <gazebo reference="caster_wheel">
         <material>Gazebo/Red</material>
+        <mu1 value="0.001"/>
+        <mu2 value="0.001"/>
     </gazebo>
     <gazebo reference="left_wheel">
@@ -15,6 +17,22 @@
     <gazebo reference="lidar">
         <material>Gazebo/Black</material>
-        <mu1 value="0.001"/>
-        <mu2 value="0.001"/>
+    </gazebo>
+    <gazebo>
+        <plugin name='diff_drive' filename='libgazebo_ros_diff_drive.so'>
+            <!-- Wheel Information -->
+            <left_joint>left_wheel_base_joint</left_joint>
+            <right_joint>right_wheel_base_joint</right_joint>
+            <wheel_separation>${chassis_width + wheel_length}</wheel_separation>
+            <wheel_diameter>${wheel_radius*2}</wheel_diameter>
+            <!-- Limits -->
+            <max_wheel_torque>200</max_wheel_torque>
+            <max_wheel_acceleration>10.0</max_wheel_acceleration>
+            <!-- Output -->
+            <odometry_frame>odom</odometry_frame>
+            <robot_base_frame>base_link</robot_base_frame>
+            <publish_odom>true</publish_odom>
+            <publish_odom_tf>true</publish_odom_tf>
+            <publish_wheel_tf>true</publish_wheel_tf>
+        </plugin>
     </gazebo>
 </robot>

File: src/my_robot/description/joints.xacro (robot description, xacro)
@@ -23,9 +23,8 @@
         <origin xyz="${chassis_length*1/5} 0 0" rpy="0 0 0"/>
     </joint>
-    <joint name="lidar_chassis_joint" type="continuous">
+    <joint name="lidar_chassis_joint" type="fixed">
         <parent link="chassis"/>
         <child link="lidar"/>
         <origin xyz="${chassis_length*7/10} 0 ${chassis_height}" rpy="0 0 0"/>
-        <axis xyz="0 0 1"/>
     </joint>
 </robot>

Commit message: add lidar, create world
add comments for launching the robot

File: src/my_robot/description/gazebo.xacro (robot description, xacro)
@@ -17,4 +17,29 @@
     <gazebo reference="lidar">
         <material>Gazebo/Black</material>
+        <sensor name="laser" type="ray">
+            <pose> 0 0 0 0 0 0 </pose>
+            <visualize>true</visualize>
+            <update_rate>10</update_rate>
+            <ray>
+                <scan>
+                    <horizontal>
+                        <samples>360</samples>
+                        <min_angle>-${pi}</min_angle>
+                        <max_angle>${pi}</max_angle>
+                    </horizontal>
+                </scan>
+                <range>
+                    <min>0.3</min>
+                    <max>12</max>
+                </range>
+            </ray>
+            <plugin name="laser_controller" filename="libgazebo_ros_ray_sensor.so">
+                <ros>
+                    <argument>~/out:=scan</argument>
+                </ros>
+                <output_type>sensor_msgs/LaserScan</output_type>
+                <frame_name>lidar</frame_name>
+            </plugin>
+        </sensor>
     </gazebo>
     <gazebo>

File: src/my_robot/description/joints.xacro (robot description, xacro)
@@ -26,5 +26,5 @@
         <parent link="chassis"/>
         <child link="lidar"/>
-        <origin xyz="${chassis_length*7/10} 0 ${chassis_height}" rpy="0 0 0"/>
+        <origin xyz="${chassis_length*7/10} 0 ${chassis_height + lidar_length/2}" rpy="0 0 0"/>
     </joint>
 </robot>

File: src/my_robot/description/links.xacro (robot description, xacro)
@@ -67,5 +67,5 @@
                 <cylinder radius="${lidar_radius}" length="${lidar_length}"/>
             </geometry>
-            <origin xyz="0 0 ${lidar_length/2}" rpy="0 0 0"/>
+            <origin xyz="0 0 0" rpy="0 0 0"/>
             <material name="black"/>
         </visual>

Commit message: separate gazebo files (lidar, control, colors)

File: src/my_robot/description/gazebo.xacro (robot description, xacro)
@@ -15,49 +15,3 @@
         <material>Gazebo/Red</material>
     </gazebo>
-    <gazebo reference="lidar">
-        <material>Gazebo/Black</material>
-        <sensor name="laser" type="ray">
-            <pose> 0 0 0 0 0 0 </pose>
-            <visualize>true</visualize>
-            <update_rate>10</update_rate>
-            <ray>
-                <scan>
-                    <horizontal>
-                        <samples>360</samples>
-                        <min_angle>-${pi}</min_angle>
-                        <max_angle>${pi}</max_angle>
-                    </horizontal>
-                </scan>
-                <range>
-                    <min>0.3</min>
-                    <max>12</max>
-                </range>
-            </ray>
-            <plugin name="laser_controller" filename="libgazebo_ros_ray_sensor.so">
-                <ros>
-                    <argument>~/out:=scan</argument>
-                </ros>
-                <output_type>sensor_msgs/LaserScan</output_type>
-                <frame_name>lidar</frame_name>
-            </plugin>
-        </sensor>
-    </gazebo>
-    <gazebo>
-        <plugin name='diff_drive' filename='libgazebo_ros_diff_drive.so'>
-            <!-- Wheel Information -->
-            <left_joint>left_wheel_base_joint</left_joint>
-            <right_joint>right_wheel_base_joint</right_joint>
-            <wheel_separation>${chassis_width + wheel_length}</wheel_separation>
-            <wheel_diameter>${wheel_radius*2}</wheel_diameter>
-            <!-- Limits -->
-            <max_wheel_torque>200</max_wheel_torque>
-            <max_wheel_acceleration>10.0</max_wheel_acceleration>
-            <!-- Output -->
-            <odometry_frame>odom</odometry_frame>
-            <robot_base_frame>base_link</robot_base_frame>
-            <publish_odom>true</publish_odom>
-            <publish_odom_tf>true</publish_odom_tf>
-            <publish_wheel_tf>true</publish_wheel_tf>
-        </plugin>
-    </gazebo>
 </robot>

File: src/my_robot/description/robot.urdf.xacro (robot description, xacro)
@@ -11,4 +11,6 @@
     <xacro:include filename="materials.xacro"/>
     <xacro:include filename="gazebo.xacro"/>
+    <xacro:include filename="gazebo_lidar.xacro"/>
+    <xacro:include filename="gazebo_control.xacro"/>
     <xacro:include filename="links.xacro"/>
     <xacro:include filename="joints.xacro"/>
