Commit message: fix wheel sliding

File: src/my_robot/description/links.xacro (robot description, xacro)
@@ -32,5 +32,5 @@
                 <xacro:insert_block name="origin"/>
                 <geometry>
-                    <cylinder radius="${wheel_radius}" length="${wheel_length}"/>
+                    <sphere radius="${wheel_radius}"/>
                 </geometry>
             </collision>
