Commit message: seperate ros2_control description for real robot and simulation

File: src/my_robot/description/robot.xacro (robot description, xacro)
@@ -2,4 +2,4 @@
 <robot name="my_robot" xmlns:xacro="http://www.ros.org/wiki/xacro">
     <xacro:include filename="components/main.xacro"/>
-    <xacro:include filename="ros2_components/main.xacro"/>
+    <xacro:include filename="ros2_components/rb_main.xacro"/>
 </robot>

File: src/my_robot/description/ros2_components/control.xacro (robot description, xacro)
@@ -1,25 +1,29 @@
 <?xml version="1.0"?>
 <robot xmlns:xacro="http://www.ros.org/wiki/xacro">
-    <ros2_control name="example_02" type="system">
+    <ros2_control name="GazeboSystem" type="system">
         <hardware>
-            <plugin>diffdrive_stm/DiffBotSystemHardware</plugin>
-            <param name="example_param_hw_start_duration_sec">0</param>
-            <param name="example_param_hw_stop_duration_sec">3.0</param>
+            <plugin>gazebo_ros2_control/GazeboSystem</plugin>
         </hardware>
-      <joint name="left_wheel_base_joint">
-        <command_interface name="velocity"/>
-        <state_interface name="position"/>
-        <state_interface name="velocity"/>
-      </joint>
-      <joint name="right_wheel_base_joint">
-        <command_interface name="velocity"/>
-        <state_interface name="position"/>
-        <state_interface name="velocity"/>
-      </joint>
+        <joint name="left_wheel_base_joint">
+            <command_interface name="velocity">
+                <param name="min">-10</param>
+                <param name="max">10</param>
+            </command_interface>
+            <state_interface name="position" />
+            <state_interface name="velocity" />
+        </joint>
+        <joint name="right_wheel_base_joint">
+            <command_interface name="velocity">
+                <param name="min">-10</param>
+                <param name="max">10</param>
+            </command_interface>
+            <state_interface name="velocity" />
+            <state_interface name="position" />
+        </joint>
     </ros2_control>
-    <!-- <gazebo>
+    <gazebo>
         <plugin filename="libgazebo_ros2_control.so" name="gazebo_ros2_control">
             <parameters>$(find my_robot)/config/my_controllers.yaml</parameters>
         </plugin>
-    </gazebo> -->
+    </gazebo>
 </robot>
