Commit message: change robot size to actual robot size

File: src/my_robot/description/components/joints.xacro (robot description, xacro)
@@ -4,5 +4,5 @@
         <parent link="base_link"/>
         <child link="chassis"/>
-        <origin xyz="-${chassis_length*7/10} 0 0"/>
+        <origin xyz="-${chassis_length*1/2} 0 0"/>
     </joint>
     <joint name="left_wheel_base_joint" type="continuous">
@@ -18,13 +18,13 @@
         <axis xyz="0 0 1"/>
     </joint>
-    <joint name="caster_wheel_chassis_joint" type="fixed">
-        <parent link="chassis"/>
+    <joint name="caster_wheel_base_joint" type="fixed">
+        <parent link="base_link"/>
         <child link="caster_wheel"/>
-        <origin xyz="${chassis_length*1/5} 0 0" rpy="0 0 0"/>
+        <origin xyz="-${caster_wheel_base_joint_length} 0 0" rpy="0 0 0"/>
     </joint>
-    <joint name="lidar_chassis_joint" type="fixed">
-        <parent link="chassis"/>
+    <joint name="lidar_base_joint" type="fixed">
+        <parent link="base_link"/>
         <child link="lidar"/>
-        <origin xyz="${chassis_length*7/10} 0 ${chassis_height + lidar_length/2}" rpy="0 0 0"/>
+        <origin xyz="0 0 ${chassis_height + lidar_length/2}" rpy="0 0 0"/>
     </joint>
 </robot>

File: src/my_robot/description/components/main.xacro (robot description, xacro)
@@ -2,10 +2,12 @@
 <robot name="my_robot" xmlns:xacro="http://www.ros.org/wiki/xacro">
     <xacro:property name="chassis_length" value="0.4"/>
-    <xacro:property name="chassis_width" value="0.3"/>
+    <xacro:property name="chassis_width" value="0.26"/>
     <xacro:property name="chassis_height" value="0.15"/>
-    <xacro:property name="wheel_radius" value="0.05"/>
-    <xacro:property name="wheel_length" value="0.03"/>
+     <!-- measured diameter is 0.68 -->
+    <xacro:property name="wheel_radius" value="0.034"/>
+    <xacro:property name="wheel_length" value="0.025"/>
     <xacro:property name="lidar_radius" value="0.05"/>
     <xacro:property name="lidar_length" value="0.03"/>
+    <xacro:property name="caster_wheel_base_joint_length" value="0.13"/>
     <xacro:include filename="inertial_macros.xacro"/>
     <xacro:include filename="materials.xacro"/>

Commit message: rotate lidar 180 degree

File: src/my_robot/description/components/joints.xacro (robot description, xacro)
@@ -26,5 +26,5 @@
         <parent link="base_link"/>
         <child link="lidar"/>
-        <origin xyz="0 0 ${chassis_height + lidar_length/2}" rpy="0 0 0"/>
+        <origin xyz="0 0 ${chassis_height + lidar_length/2}" rpy="0 0 ${pi}"/>
     </joint>
 </robot>

Commit message: change chassis, caster

File: src/my_robot/description/components/joints.xacro (robot description, xacro)
@@ -4,10 +4,10 @@
         <parent link="base_link"/>
         <child link="chassis"/>
-        <origin xyz="-${chassis_length*1/2} 0 0"/>
+        <origin xyz="0 0 ${chassis_height/2}"/>
     </joint>
     <joint name="left_wheel_base_joint" type="continuous">
         <parent link="base_link"/>
         <child link="left_wheel"/>
-        <origin xyz="0 ${chassis_width/2 + wheel_length/2} 0" rpy="-${pi/2} 0 0"/>
+        <origin xyz="0 ${chassis_radius - wheel_length/2} 0" rpy="-${pi/2} 0 0"/>
         <axis xyz="0 0 1"/>
     </joint>
@@ -15,11 +15,16 @@
         <parent link="base_link"/>
         <child link="right_wheel"/>
-        <origin xyz="0 -${chassis_width/2 + wheel_length/2} 0" rpy="-${pi/2} 0 0"/>
+        <origin xyz="0 -${chassis_radius - wheel_length/2} 0" rpy="-${pi/2} 0 0"/>
         <axis xyz="0 0 1"/>
     </joint>
-    <joint name="caster_wheel_base_joint" type="fixed">
+    <joint name="caster_box_base_joint" type="fixed">
         <parent link="base_link"/>
+        <child link="caster_box"/>
+        <origin xyz="${caster_wheel_base_joint_length} 0 -${(wheel_radius - caster_wheel_radius)/2}" rpy="0 0 0"/>
+    </joint>
+    <joint name="caster_box_caster_wheel_joint" type="fixed">
+        <parent link="caster_box"/>
         <child link="caster_wheel"/>
-        <origin xyz="-${caster_wheel_base_joint_length} 0 0" rpy="0 0 0"/>
+        <origin xyz="0 0 -${(wheel_radius - caster_wheel_radius)/2}" rpy="0 0 0"/>
     </joint>
     <joint name="lidar_base_joint" type="fixed">

File: src/my_robot/description/components/links.xacro (robot description, xacro)
@@ -4,19 +4,19 @@
     <link name="chassis">
         <visual>
-            <origin xyz="${chassis_length/2} 0 ${chassis_height/2}" rpy="0 0 0"/>
+            <origin xyz="0 0 0" rpy="0 0 0"/>
             <geometry>
-                <box size="${chassis_length} ${chassis_width} ${chassis_height}"/>
+                <cylinder radius="${chassis_radius}" length="${chassis_height}"/>
             </geometry>
             <material name="white"/>
         </visual>
         <collision>
-            <origin xyz="${chassis_length/2} 0 ${chassis_height/2}" rpy="0 0 0"/>
+            <origin xyz="0 0 0" rpy="0 0 0"/>
             <geometry>
-                <box size="${chassis_length} ${chassis_width} ${chassis_height}"/>
+                <cylinder radius="${chassis_radius}" length="${chassis_height}"/>
             </geometry>
         </collision>
-        <xacro:inertial_box mass="0.5" x="${chassis_length}" y="${chassis_width}" z="${chassis_height}">
-            <origin xyz="${chassis_length/2} 0 ${chassis_height/2}" rpy="0 0 0"/>
-        </xacro:inertial_box>
+        <xacro:inertial_cylinder mass="0.5" length="${chassis_height}" radius="${chassis_radius}">
+            <origin xyz="${chassis_radius/2} 0 0" rpy="0 0 0"/>
+        </xacro:inertial_cylinder>
     </link>
     <xacro:macro name="wheel" params="name *origin">
@@ -49,5 +49,5 @@
         <visual>
             <geometry>
-                <sphere radius="${wheel_radius}"/>
+                <sphere radius="${caster_wheel_radius}"/>
             </geometry>
             <material name="red"/>
@@ -55,10 +55,25 @@
         <collision>
             <geometry>
-                <sphere radius="${wheel_radius}"/>
+                <sphere radius="${caster_wheel_radius}"/>
             </geometry>
         </collision>
-        <xacro:inertial_sphere mass="0.1" radius="${wheel_radius}">
+        <xacro:inertial_sphere mass="0.001" radius="${caster_wheel_radius}">
             <origin xyz="0 0 0" rpy="0 0 0"/>
         </xacro:inertial_sphere>
+    </link>
+    <link name="caster_box">
+        <visual>
+            <geometry>
+                <box size="${2*caster_wheel_radius} ${2*caster_wheel_radius} ${wheel_radius - caster_wheel_radius}"/>
+            </geometry>
+        </visual>
+        <collision>
+            <geometry>
+                <box size="${2*caster_wheel_radius} ${2*caster_wheel_radius} ${wheel_radius - caster_wheel_radius}"/>
+            </geometry>
+        </collision>
+        <xacro:inertial_box mass="0.01" x="${2*caster_wheel_radius}" y="${2*caster_wheel_radius}" z="${wheel_radius - caster_wheel_radius}">
+            <origin xyz="0 0 0" rpy="0 0 0"/>
+        </xacro:inertial_box>
     </link>
     <link name="lidar">

File: src/my_robot/description/components/main.xacro (robot description, xacro)
@@ -1,13 +1,13 @@
 <?xml version="1.0"?>
 <robot name="my_robot" xmlns:xacro="http://www.ros.org/wiki/xacro">
-    <xacro:property name="chassis_length" value="0.4"/>
-    <xacro:property name="chassis_width" value="0.26"/>
-    <xacro:property name="chassis_height" value="0.15"/>
+    <xacro:property name="chassis_radius" value="0.15"/>
+    <xacro:property name="chassis_height" value="0.067"/>
      <!-- measured diameter is 0.68 -->
     <xacro:property name="wheel_radius" value="0.034"/>
     <xacro:property name="wheel_length" value="0.025"/>
-    <xacro:property name="lidar_radius" value="0.05"/>
-    <xacro:property name="lidar_length" value="0.03"/>
+    <xacro:property name="lidar_radius" value="0.035"/>
+    <xacro:property name="lidar_length" value="0.024"/>
     <xacro:property name="caster_wheel_base_joint_length" value="0.13"/>
+    <xacro:property name="caster_wheel_radius" value="0.006"/>
     <xacro:include filename="inertial_macros.xacro"/>
     <xacro:include filename="materials.xacro"/>
